File: kiCad/esp32_Keyboard/esp32_Keyboard.kicad_pcb (KiCad board)
At the start: 2 copper layers, 171 parts, among them SW1 Switch, SW10 Switch, SW11 Switch, SW12 Switch, SW13 Switch, SW14 Switch, SW15 Switch, SW16 Switch, SW17 Switch, SW18 Switch, SW19 Switch, SW2 Switch, SW20 Switch, SW21 Switch, SW22 Switch, SW23 Switch, SW24 Switch, SW25 Switch, SW26 Switch, SW27 Switch, SW28 Switch, SW29 Switch, SW3 Switch, SW30 Switch, SW31 Switch, SW32 Switch, SW33 Switch, SW34 Switch, SW35 Switch, SW36 Switch, SW37 Switch, SW38 Switch, SW39 Switch, SW4 Switch, SW40 Switch, SW41 Switch, SW42 Switch, SW43 Switch, SW44 Switch, SW45 Switch, SW46 Switch, SW47 Switch, SW48 Switch, SW49 Switch, SW5 Switch, SW50 Switch, SW51 Switch, SW52 Switch, SW53 Switch, SW54 Switch, SW55 Switch, SW56 Switch, SW57 Switch, SW58 Switch, SW59 Switch, SW6 Switch, SW60 Switch, SW61 Switch, SW62 Switch, SW63 Switch, SW64 Switch, SW65 Switch, SW66 Switch, SW67 Switch, SW68 Switch, SW69 Switch, SW7 Switch, SW70 Switch, SW71 Switch, SW72 Switch, SW73 Switch, SW74 Switch, SW75 Switch, SW76 Switch, SW77 Switch, SW78 Switch, SW79 Switch, SW8 Switch, SW80 Switch, SW81 Switch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

Commit message: finished layout circuit baord V1
Parts:
- added Dsp1: ~, tigmitLib:GC9A01 roundDisplay Footprint, F.Cu at (351.6, 88.9)
- added J1: Conn_01x15, Connector_PinHeader_2.54mm:PinHeader_1x15_P2.54mm_Vertical, F.Cu at (10.3, 25.9)
- added J2: Conn_01x15, Connector_PinHeader_2.54mm:PinHeader_1x15_P2.54mm_Vertical, F.Cu at (-31.0, 61.3)
- added R2: 10K, Resistor_THT:R_Axial_DIN0204_L3.6mm_D1.6mm_P7.62mm_Horizontal, B.Cu at (13.7, 61.9)
- added R3: 10K, Resistor_THT:R_Axial_DIN0204_L3.6mm_D1.6mm_P7.62mm_Horizontal, B.Cu at (7.94, 74.8)
- added R4: 10K, Resistor_THT:R_Axial_DIN0204_L3.6mm_D1.6mm_P7.62mm_Horizontal, B.Cu at (7.94, 93.8)
- added R5: 10K, Resistor_THT:R_Axial_DIN0204_L3.6mm_D1.6mm_P7.62mm_Horizontal, B.Cu at (7.94, 112.9)
- added R6: 10K, Resistor_THT:R_Axial_DIN0204_L3.6mm_D1.6mm_P7.62mm_Horizontal, B.Cu at (7.94, 132.7)
- added R7: 10K, Resistor_THT:R_Axial_DIN0204_L3.6mm_D1.6mm_P7.62mm_Horizontal, B.Cu at (7.94, 151.0)
- added U4: ~, tigmitLib:b103 multichannel fader pot, F.Cu at (-3.17, 115.9)
- added U5: ESP32-DEVKIT-V1 DisplayHandler, ESP32-DEVKIT-V1:MODULE_ESP32_DEVKIT_V1, F.Cu at (346.1, 36.5)
- R1: footprint ScottoKeebs_Components:Resistor_0402 -> Resistor_THT:R_Axial_DIN0204_L3.6mm_D1.6mm_P7.62mm_Horizontal
- SW1, SW10, SW11, SW12, SW13, SW14, SW15, SW16, SW17, SW18, SW19, SW2, SW20, SW21, SW22, SW23, SW24, SW25, SW26, SW27, SW29, SW3, SW31, SW32, SW33, SW34, SW35, SW36, SW37, SW38, SW39, SW4, SW40, SW41, SW42, SW44, SW46, SW47, SW48, SW49, SW5, SW50, SW51, SW52, SW53, SW54, SW55, SW56, SW59, SW6, SW60, SW61, SW62, SW63, SW64, SW65, SW66, SW67, SW68, SW7, SW70, SW79, SW8, SW80, SW81, SW9: footprint ScottoKeebs_MX:MX_PCB_1.00u -> ScottoKeebs_Hotswap:Hotswap_MX_1.00u
- SW28: footprint ScottoKeebs_MX:MX_PCB_2.00u -> ScottoKeebs_Hotswap:Hotswap_MX_2.00u
- SW30, SW43: footprint ScottoKeebs_MX:MX_PCB_1.50u -> ScottoKeebs_Hotswap:Hotswap_MX_1.50u
- SW45: footprint ScottoKeebs_MX:MX_PCB_1.75u -> ScottoKeebs_Hotswap:Hotswap_MX_1.75u
- SW57, SW58: footprint ScottoKeebs_MX:MX_PCB_2.25u -> ScottoKeebs_Hotswap:Hotswap_MX_2.25u
- SW69: footprint ScottoKeebs_MX:MX_PCB_2.75u -> ScottoKeebs_Hotswap:Hotswap_MX_2.75u
- SW71, SW72, SW73, SW75, SW76, SW77, SW78: footprint ScottoKeebs_MX:MX_PCB_1.25u -> ScottoKeebs_Hotswap:Hotswap_MX_1.25u
- SW74: footprint ScottoKeebs_MX:MX_PCB_6.25u -> ScottoKeebs_Hotswap:Hotswap_MX_6.25u
- U1: value ESP32-DEVKIT-V1 -> ESP32-DEVKIT-V1 Matrix Handler
- moved U1 47.8 mm to (-10.3, 41.3)
- moved D42 14.6 mm to (263.4, 85.2), turned to 120 degrees
- moved D43 12.7 mm to (287.2, 86.2), turned to 120 degrees
- moved R1 11.9 mm to (42.9, 12.1)
- moved D13 9.53 mm to (295.1, 37.6), turned to 120 degrees
- moved D14 9.53 mm to (318.9, 37.6), turned to 120 degrees
- moved D29 9.53 mm to (318.9, 66.2), turned to 120 degrees
- moved D44 9.53 mm to (318.9, 85.2), turned to 120 degrees
- moved D57 9.53 mm to (283.2, 104.3), turned to 120 degrees
- moved D69 9.53 mm to (278.4, 123.3), turned to 120 degrees
- moved D70 9.53 mm to (338.0, 123.3), turned to 120 degrees
- moved D79 9.53 mm to (318.9, 142.4), turned to 120 degrees
- moved D80 9.53 mm to (338.0, 142.4), turned to 120 degrees
- moved D10 9.53 mm to (238.0, 37.6), turned to 120 degrees
- moved D17 9.53 mm to (66.5, 66.2), turned to 120 degrees
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Connections:
- U1 pad 1: VCC -> /SRCLR
- U1 pad 10: RCLK -> Net-(J2-Pin_6)
- U1 pad 11: SER -> esp32-SDA
- U1 pad 12: unconnected-(U1-RX0-Pad12) -> Net-(J2-Pin_4)
- U1 pad 13: unconnected-(U1-TX0-Pad13) -> Net-(J2-Pin_3)
- U1 pad 14: Row5 -> DSP CS
- U1 pad 15: Row4 -> SER / DATA
- U1 pad 16: unconnected-(U1-EN-Pad16) -> Net-(J1-Pin_15)
- U1 pad 17: unconnected-(U1-VP-Pad17) -> Net-(J1-Pin_14)
- U1 pad 18: unconnected-(U1-VN-Pad18) -> Net-(J1-Pin_13)
- U1 pad 19: unconnected-(U1-D34-Pad19) -> Row0
- U1 pad 2: GND -> /OE
- U1 pad 20: unconnected-(U1-D35-Pad20) -> Row1
- U1 pad 21: Row0 -> Row2
- U1 pad 22: unconnected-(U1-D33-Pad22) -> Row3
- U1 pad 23: Row3 -> Row4
- U1 pad 24: Row2 -> Row5
- U1 pad 25: Row1 -> Net-(J1-Pin_6)
- U1 pad 26: unconnected-(U1-D14-Pad26) -> Net-(J1-Pin_5)
- U1 pad 27: unconnected-(U1-D12-Pad27) -> Net-(J1-Pin_4)
- U1 pad 28: unconnected-(U1-D13-Pad28) -> RCLK / LATCH
- U1 pad 29: GND -> /OE
- U1 pad 3: /OE -> Net-(J2-Pin_13)
- U1 pad 30: unconnected-(U1-VIN-Pad30) -> Net-(J1-Pin_1)
- U1 pad 4: unconnected-(U1-D2-Pad4) -> Net-(J2-Pin_12)
- U1 pad 5: unconnected-(U1-D4-Pad5) -> Net-(J2-Pin_11)
- U1 pad 6: unconnected-(U1-RX2-Pad6) -> Net-(J2-Pin_10)
- U1 pad 7: unconnected-(U1-TX2-Pad7) -> Net-(J2-Pin_9)
- U1 pad 8: unconnected-(U1-D5-Pad8) -> Net-(J2-Pin_8)
- U1 pad 9: /SRCLR -> SRCLK / CLOCK
- U2 pad 11: RCLK -> SRCLK / CLOCK
- U2 pad 12: RCLK -> RCLK / LATCH
- U2 pad 14: SER -> SER / DATA
- U2 pad 16: VCC -> /SRCLR
- U2 pad 8: GND -> /OE
- U3 pad 11: RCLK -> SRCLK / CLOCK
- U3 pad 12: RCLK -> RCLK / LATCH
- U3 pad 16: VCC -> /SRCLR
- U3 pad 8: GND -> /OE
Routing:
- net /SRCLR: track 163.1 -> 606.5 mm, vias 1 -> 0
- net RCLK: track 164.3 -> 0.00 mm
- net (no net): track 0.00 -> 164.3 mm
- net VCC: track 161.0 -> 0.00 mm
- net Row4: track 297.7 -> 430.7 mm, vias 0 -> 2
- net Row1: track 290.5 -> 410.3 mm, vias 0 -> 15
- net Row2: track 285.8 -> 398.7 mm, vias 0 -> 15
- net DSP RST: track 0.00 -> 96.1 mm
- net Row0: track 290.5 -> 382.1 mm, vias 0 -> 14
- net Row3: track 348.7 -> 437.2 mm, vias 0 -> 13
- net DSP DC: track 0.00 -> 84.3 mm
- net DSP SCL: track 0.00 -> 79.7 mm
- net Row5: track 307.2 -> 384.1 mm
- net DSP CS: track 0.00 -> 76.3 mm
- net DSP  SDA: track 0.00 -> 74.0 mm
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
Commit message: finished PCB design
Parts:
- removed J1, J2: Conn_01x15, Connector_PinHeader_2.54mm:PinHeader_1x15_P2.54mm_Vertical
- removed R1: 10K, Resistor_THT:R_Axial_DIN0204_L3.6mm_D1.6mm_P7.62mm_Horizontal
- Dsp1: footprint tigmitLib:GC9A01 roundDisplay Footprint -> Connector_PinHeader_2.54mm:PinHeader_1x07_P2.54mm_Vertical; moved to B.Cu
- U1, U2, U3, U5: moved to B.Cu
- moved U2 111.2 mm to (132.6, 51.4), turned to 0 degrees
- moved U3 48.2 mm to (218.3, 51.4), turned to 0 degrees
- moved R2 43.6 mm to (53.2, 43.5), turned to 90 degrees
- moved U5 39.7 mm to (314.3, 60.3), turned to 180 degrees
- moved U1 33.6 mm to (22.7, 47.6), turned to -90 degrees
- moved Dsp1 21.6 mm to (330.2, 91.3)
- moved U4 5.32 mm to (-0.79, 111.1)
- moved R4 3.19 mm to (11.1, 93.5), turned to 90 degrees
- moved R5 3.19 mm to (11.1, 112.6), turned to 90 degrees
- moved R3 3.19 mm to (11.1, 74.5), turned to 90 degrees
- moved R6 3.19 mm to (11.1, 132.4), turned to 90 degrees
- moved R7 3.19 mm to (11.1, 150.7), turned to 90 degrees
- moved D1 2.84 mm to (31.0, 38.9), turned to 0 degrees
- moved D6 1.42 mm to (151.6, 38.9), turned to 180 degrees
- moved D9 1.42 mm to (208.8, 38.9), turned to 180 degrees
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Connections:
- U1 pad 10: Net-(J2-Pin_6) -> unconnected-(U1-D19-Pad10)
- U1 pad 12: Net-(J2-Pin_4) -> unconnected-(U1-RX0-Pad12)
- U1 pad 13: Net-(J2-Pin_3) -> unconnected-(U1-TX0-Pad13)
- U1 pad 16: Net-(J1-Pin_15) -> unconnected-(U1-EN-Pad16)
- U1 pad 17: Net-(J1-Pin_14) -> unconnected-(U1-VP-Pad17)
- U1 pad 18: Net-(J1-Pin_13) -> unconnected-(U1-VN-Pad18)
- U1 pad 25: Net-(J1-Pin_6) -> unconnected-(U1-D27-Pad25)
- U1 pad 26: Net-(J1-Pin_5) -> unconnected-(U1-D14-Pad26)
- U1 pad 27: Net-(J1-Pin_4) -> POT slider Pin
- U1 pad 3: Net-(J2-Pin_13) -> unconnected-(U1-D15-Pad3)
- U1 pad 30: Net-(J1-Pin_1) -> unconnected-(U1-VIN-Pad30)
- U1 pad 4: Net-(J2-Pin_12) -> unconnected-(U1-D2-Pad4)
- U1 pad 5: Net-(J2-Pin_11) -> unconnected-(U1-D4-Pad5)
- U1 pad 6: Net-(J2-Pin_10) -> unconnected-(U1-RX2-Pad6)
- U1 pad 7: Net-(J2-Pin_9) -> unconnected-(U1-TX2-Pad7)
- U1 pad 8: Net-(J2-Pin_8) -> unconnected-(U1-D5-Pad8)
Routing:
- net esp32-SDA: track 0.00 -> 389.9 mm
- net DSP CS: track 76.3 -> 354.2 mm
- net RCLK / LATCH: track 0.00 -> 255.1 mm, vias 0 -> 4
- net SRCLK / CLOCK: track 0.00 -> 242.1 mm, vias 0 -> 2
- net (no net): track 164.3 -> 0.00 mm
- net /OE: track 184.9 -> 40.5 mm, vias 0 -> 2
- net SER / DATA: track 0.00 -> 115.4 mm, vias 0 -> 1
- net Col6: track 237.9 -> 130.4 mm, vias 0 -> 3
- net Row5: track 384.1 -> 487.1 mm
- net Row4: track 430.7 -> 528.1 mm, vias 2 -> 3
- net Col5: track 242.6 -> 162.7 mm
- net Col0: track 172.2 -> 249.6 mm, vias 0 -> 1
- net Col7: track 257.6 -> 186.8 mm
- net Row3: track 437.2 -> 506.3 mm
- net Col15: track 280.0 -> 226.6 mm, vias 0 -> 3
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- added copper zone on B.Cu, net /OE
- added copper zone on F.Cu, net /OE
Other:
- board outline added: 376.2 x 139.7 mm

Commit message: commit current work
Parts:
- added BT1: Battery_Cell, tigmitLib:battery solder pins, F.Cu at (358.0, 78.6)
- added C1: 100µF, Capacitor_THT:CP_Radial_D10.0mm_P2.50mm, F.Cu at (413.5, 73.8)
- added C2: 100nF, Capacitor_THT:C_Rect_L7.0mm_W2.5mm_P5.00mm, F.Cu at (403.9, 73.6)
- added R1: 4k7, Resistor_THT:R_Axial_DIN0204_L3.6mm_D1.6mm_P7.62mm_Horizontal, F.Cu at (417.5, 91.4)
- added R10: 100k, Resistor_THT:R_Axial_DIN0204_L3.6mm_D1.6mm_P7.62mm_Horizontal, F.Cu at (412.6, 84.1)
- added R8: 10k, Resistor_THT:R_Axial_DIN0204_L3.6mm_D1.6mm_P7.62mm_Horizontal, F.Cu at (415.1, 109.4)
- added R9: 100k, Resistor_THT:R_Axial_DIN0204_L3.6mm_D1.6mm_P7.62mm_Horizontal, F.Cu at (405.0, 81.0)
- added U6: SK12D07VG4, SK12D07VG4:SK12D07VG4, B.Cu at (331.8, 70.6)
- added mcp1: ~, tigmitLib:MCP1700 3.3V, F.Cu at (392.1, 74.6)
- Dsp1, R2, R3, R4, R5, R6, R7: moved to F.Cu
- S1: value stab L shift 2.25u -> stab space 6.25u; footprint PCM_marbastlib-mx:STAB_MX_2.25u -> PCM_marbastlib-mx:STAB_MX_6.25u
- S2: value stab space 6.25u -> stab 2u; footprint PCM_marbastlib-mx:STAB_MX_6.25u -> PCM_marbastlib-mx:STAB_MX_2u
- S3: value stab R shift 2.75u -> stab 2u; footprint PCM_marbastlib-mx:STAB_MX_2.75u -> PCM_marbastlib-mx:STAB_MX_2u
- S4: value stab enter 2.25u -> stab 2u; footprint PCM_marbastlib-mx:STAB_MX_2.25u -> PCM_marbastlib-mx:STAB_MX_2u
- S5: value stab backspace 2u -> stab 2u
- U1: footprint ESP32-DEVKIT-V1:MODULE_ESP32_DEVKIT_V1 -> tigmitLib:ESP32 Vroom Devkit V1; moved to F.Cu
- U2, U3: footprint SN74HC595NG4:DIP794W45P254L1969H508Q16 -> tigmitLib:SNH Shift register
- U5: value ESP32-DEVKIT-V1 DisplayHandler -> ~; footprint ESP32-DEVKIT-V1:MODULE_ESP32_DEVKIT_V1 -> tp4056:TP4056-18650
- moved S1 479.6 mm to (473.1, 331.0)
- moved R5 403.8 mm to (414.3, 91.4), turned to -90 degrees
- moved R7 403.0 mm to (412.0, 109.4)
- moved R4 399.3 mm to (410.4, 91.4), turned to -90 degrees
- moved R6 398.3 mm to (408.8, 109.4)
- moved R3 395.7 mm to (406.4, 91.4), turned to -90 degrees
- moved U1 391.6 mm to (409.8, 106.9), turned to 0 degrees
- moved S2 363.3 mm to (498.0, 239.7)
- moved R2 352.5 mm to (402.4, 91.4), turned to -90 degrees
- moved S5 311.5 mm to (498.0, 300.6)
- moved S4 274.6 mm to (498.0, 280.3)
- moved U2 267.2 mm to (375.5, 162.6), turned to -90 degrees
- moved S3 257.0 mm to (498.0, 260.0)
- moved U3 183.4 mm to (375.5, 145.9), turned to -90 degrees
- moved Dsp1 103.8 mm to (414.3, 152.1)
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Connections:
- Dsp1 pad 3: DSP SCL -> DP_SCL
- Dsp1 pad 4: DSP  SDA -> DP_SDA
- Dsp1 pad 5: DSP DC -> DP_DC
- Dsp1 pad 6: DSP CS -> DP_CS
- Dsp1 pad 7: DSP RST -> DP_RST
- U1 pad 14: DSP CS -> esp32-SCL
- U1 pad 25: unconnected-(U1-D27-Pad25) -> batt_voltage_Pin
- U1 pad 26: unconnected-(U1-D14-Pad26) -> batt_chargesense
- U1 pad 3: unconnected-(U1-D15-Pad3) -> DP_CS
- U1 pad 4: unconnected-(U1-D2-Pad4) -> DP_DC
- U1 pad 5: unconnected-(U1-D4-Pad5) -> DP_SDA
- U1 pad 8: unconnected-(U1-D5-Pad8) -> DP_RST
- U1 pad 9: SRCLK / CLOCK -> DP_SCL
- U2 pad 11: SRCLK / CLOCK -> DP_SCL
- U3 pad 11: SRCLK / CLOCK -> DP_SCL
- U5 pad 1: /SRCLR -> Net-(U5-ind)
- U5 pad 3: unconnected-(U5-D15-Pad3) -> Net-(U5-OUT+)
- U5 pad 4: unconnected-(U5-D2-Pad4) -> /OE
- U5 pad 5: DSP RST -> Net-(U5-B+)
- U5 pad 6: DSP DC -> Battery-
Routing:
- net esp32-SDA: track 389.9 -> 0.00 mm
- net DSP CS: track 354.2 -> 0.00 mm
- net /SRCLR: track 576.3 -> 312.5 mm, vias 3 -> 0
- net /OE: track 40.5 -> 289.7 mm, vias 2 -> 3
- net SRCLK / CLOCK: track 242.1 -> 0.00 mm, vias 2 -> 0
- net RCLK / LATCH: track 255.1 -> 100.6 mm, vias 4 -> 0
- net Col1: track 184.2 -> 329.2 mm
- net Col15: track 226.6 -> 86.1 mm, vias 3 -> 2
- net Col14: track 254.0 -> 122.2 mm, vias 1 -> 0
- net Col0: track 249.6 -> 380.5 mm
- net Col4: track 162.5 -> 283.4 mm, vias 0 -> 1
- net Col6: track 130.4 -> 250.3 mm, vias 3 -> 1
- net Col5: track 162.7 -> 279.8 mm, vias 0 -> 1
- net Col3: track 186.7 -> 298.8 mm, vias 0 -> 1
- net Col2: track 238.2 -> 336.2 mm, vias 0 -> 1
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- removed copper zone on B.Cu, net /OE
- removed copper zone on F.Cu, net /OE
Other:
- board outline removed

Commit message: added ecoder and LED Support
Parts:
- added C3: 100µF, Capacitor_THT:CP_Radial_D10.0mm_P2.50mm, F.Cu at (459.4, 178.3)
- added C4: 100µF, Capacitor_THT:CP_Radial_D10.0mm_P2.50mm, F.Cu at (459.4, 189.9)
- added R11: 10k, Resistor_THT:R_Axial_DIN0204_L3.6mm_D1.6mm_P7.62mm_Horizontal, F.Cu at (467.9, 191.7)
- added SW82: ~, tigmitLib:hotswap socket with neopixel, F.Cu at (475.3, 180.3)
Connections:
- U1 pad 10: unconnected-(U1-D19-Pad10) -> NEOPIXEL_CONTROLL
Other:
- board outline added: 523.1 x 307.2 mm
