File: kiCad/esp32_Keyboard/esp32_Keyboard.kicad_sch (KiCad schematic)
At the start: 188 parts, among them SW1 Switch, SW10 Switch, SW11 Switch, SW12 Switch, SW13 Switch, SW14 Switch, SW15 Switch, SW16 Switch, SW17 Switch, SW18 Switch, SW19 Switch, SW2 Switch, SW20 Switch, SW21 Switch, SW22 Switch, SW23 Switch, SW24 Switch, SW25 Switch, SW26 Switch, SW27 Switch, SW28 Switch, SW29 Switch, SW3 Switch, SW30 Switch, SW31 Switch, SW32 Switch, SW33 Switch, SW34 Switch, SW35 Switch, SW36 Switch, SW37 Switch, SW38 Switch, SW39 Switch, SW4 Switch, SW40 Switch, SW41 Switch, SW42 Switch, SW43 Switch, SW44 Switch, SW45 Switch, SW46 Switch, SW47 Switch, SW48 Switch, SW49 Switch, SW5 Switch, SW50 Switch, SW51 Switch, SW52 Switch, SW53 Switch, SW54 Switch, SW55 Switch, SW56 Switch, SW57 Switch, SW58 Switch, SW59 Switch, SW6 Switch, SW60 Switch, SW61 Switch, SW62 Switch, SW63 Switch, SW64 Switch, SW65 Switch, SW66 Switch, SW67 Switch, SW68 Switch, SW69 Switch, SW7 Switch, SW70 Switch, SW71 Switch, SW72 Switch, SW73 Switch, SW74 Switch, SW75 Switch, SW76 Switch, SW77 Switch, SW78 Switch, SW79 Switch, SW8 Switch, SW80 Switch, SW81 Switch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

Commit message: added ecoder and LED Support
Parts:
- added C3, C4: 100µF, Capacitor_THT:CP_Radial_D10.0mm_P2.50mm, symbol Device:C_Polarized
- added R11: 10k, Resistor_THT:R_Axial_DIN0204_L3.6mm_D1.6mm_P7.62mm_Horizontal, symbol ScottoKeebs:Placeholder_Resistor
- added SW82: ~, tigmitLib:hotswap socket with neopixel, symbol tigmitSymbolLib:Switch_+_LED
Connections:
- net GND: now also C3.2, C4.2, R11.2
- net RCLK / LATCH: now also R11.1
- net VCC: now also C3.1, C4.1
Other:
- moved on the sheet: BT1, C1, C2, R1, R10, R8, R9, U2, U3, U4, U5, U6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

Commit message: saving kicad progress HW rev2
Parts:
- removed BT1: Battery_Cell, tigmitLib:battery solder pins, symbol Device:Battery_Cell
- removed C1: 100µF, Capacitor_THT:CP_Radial_D10.0mm_P2.50mm, symbol Device:C_Polarized
- removed C2: 100nF, Capacitor_THT:C_Rect_L7.0mm_W2.5mm_P5.00mm, symbol Device:C
- removed D80, D81: Diode, ScottoKeebs_Components:Diode_SOD-123, symbol ScottoKeebs:Placeholder_Diode
- removed R1: 4k7, Resistor_THT:R_Axial_DIN0204_L3.6mm_D1.6mm_P7.62mm_Horizontal, symbol ScottoKeebs:Placeholder_Resistor
- removed R10, R9: 100k, Resistor_THT:R_Axial_DIN0204_L3.6mm_D1.6mm_P7.62mm_Horizontal, symbol ScottoKeebs:Placeholder_Resistor
- removed R8: 10k, Resistor_THT:R_Axial_DIN0204_L3.6mm_D1.6mm_P7.62mm_Horizontal, symbol ScottoKeebs:Placeholder_Resistor
- removed S2: stab 2u, PCM_marbastlib-mx:STAB_MX_2u, symbol PCM_marbastlib-mx:MX_stab
- removed SW1, SW10, SW11, SW12, SW13, SW14, SW15, SW16, SW17, SW18, SW19, SW2, SW20, SW21, SW22, SW23, SW24, SW25, SW26, SW27, SW29, SW3, SW31, SW32, SW33, SW34, SW35, SW36, SW37, SW38, SW39, SW4, SW40, SW41, SW42, SW44, SW46, SW47, SW48, SW49, SW5, SW50, SW51, SW52, SW53, SW54, SW55, SW56, SW59, SW6, SW60, SW61, SW62, SW63, SW64, SW65, SW66, SW67, SW68, SW7, SW70, SW79, SW8, SW80, SW81, SW9: Switch, ScottoKeebs_Hotswap:Hotswap_MX_1.00u, symbol ScottoKeebs:Placeholder_Switch
- removed SW28: Switch, ScottoKeebs_Hotswap:Hotswap_MX_2.00u, symbol ScottoKeebs:Placeholder_Switch
- removed SW30, SW43: Switch, ScottoKeebs_Hotswap:Hotswap_MX_1.50u, symbol ScottoKeebs:Placeholder_Switch
- removed SW45: Switch, ScottoKeebs_Hotswap:Hotswap_MX_1.75u, symbol ScottoKeebs:Placeholder_Switch
- removed SW57, SW58: Switch, ScottoKeebs_Hotswap:Hotswap_MX_2.25u, symbol ScottoKeebs:Placeholder_Switch
- removed SW69: Switch, ScottoKeebs_Hotswap:Hotswap_MX_2.75u, symbol ScottoKeebs:Placeholder_Switch
- removed SW71, SW72, SW73, SW75, SW76, SW77, SW78: Switch, ScottoKeebs_Hotswap:Hotswap_MX_1.25u, symbol ScottoKeebs:Placeholder_Switch
- removed SW74: Switch, ScottoKeebs_Hotswap:Hotswap_MX_6.25u, symbol ScottoKeebs:Placeholder_Switch
- removed SW82: ~, tigmitLib:hotswap socket with neopixel, symbol tigmitSymbolLib:Switch_+_LED
- removed U5: ~, tp4056:TP4056-18650, symbol tigmitSymbolLib:tp_lipo_chargin_module
- removed U6: SK12D07VG4, SK12D07VG4:SK12D07VG4, symbol SK12D07VG4:SK12D07VG4
- removed mcp1: ~, tigmitLib:MCP1700 3.3V, symbol tigmitSymbolLib:tim_mcp1700-3302e
- added PWR_Module1: Conn_01x04_Pin, Connector_PinHeader_2.54mm:PinHeader_1x04_P2.54mm_Vertical, symbol Connector:Conn_01x04_Pin
- added RotaryEnc1: Conn_01x05_Pin, Connector_PinHeader_2.54mm:PinHeader_1x05_P2.54mm_Vertical, symbol Connector:Conn_01x05_Pin
- added SW1, SW10, SW11, SW12, SW13, SW14, SW15, SW16, SW17, SW18, SW19, SW2, SW20, SW21, SW22, SW23, SW24, SW25, SW26, SW27, SW28, SW29, SW3, SW30, SW31, SW32, SW33, SW34, SW35, SW36, SW37, SW38, SW39, SW4, SW40, SW41, SW42, SW43, SW44, SW45, SW46, SW47, SW48, SW49, SW5, SW50, SW51, SW52, SW53, SW54, SW55, SW56, SW57, SW58, SW59, SW6, SW60, SW61, SW62, SW63, SW64, SW65, SW66, SW67, SW68, SW69, SW7, SW70, SW71, SW72, SW73, SW74, SW75, SW76, SW77, SW78, SW79, SW8, SW9: ~, tigmitLib:hotswap socket with neopixel, symbol tigmitSymbolLib:Switch_+_LED
- added U3: BOB-12009, BOB-12009:CONV_BOB-12009, symbol BOB-12009:BOB-12009
- C1: renamed from C4; footprint Capacitor_THT:CP_Radial_D10.0mm_P2.50mm -> Capacitor_SMD:CP_Elec_6.3x5.2
- C2: renamed from C3; footprint Capacitor_THT:CP_Radial_D10.0mm_P2.50mm -> Capacitor_SMD:CP_Elec_6.3x5.2
- renumbered R11 to R1, S3 to S1, S4 to S2, S5 to S3, S1 to S4, U2 to U1, U3 to U2, U1 to U5
Connections:
- net Col0: now also D13.2 (A), D28.2 (A), D43.2 (A), D57.2 (A), D70.2 (A); no longer D15.2 (A), D30.2 (A), D45.2 (A), D58.2 (A), D71.2 (A)
- net Col1: now also D14.2 (A), D29.2 (A), D44.2 (A), D71.2 (A); no longer D16.2 (A), D31.2 (A), D46.2 (A), D59.2 (A), D72.2 (A)
- net Col10: now also D23.2 (A), D38.2 (A), D53.2 (A), D66.2 (A), D75.2 (A), D9.2 (A); no longer D10.2 (A), D25.2 (A), D40.2 (A), D55.2 (A), D68.2 (A), D76.2 (A)
- net Col11: now also D10.2 (A), D24.2 (A), D39.2 (A), D54.2 (A), D67.2 (A), D76.2 (A); no longer D11.2 (A), D26.2 (A), D41.2 (A), D56.2 (A), D77.2 (A)
- net Col12: now also D11.2 (A), D25.2 (A), D40.2 (A), D68.2 (A), D77.2 (A); no longer D12.2 (A), D27.2 (A), D42.2 (A), D69.2 (A), D78.2 (A)
- net Col13: now also D12.2 (A), D26.2 (A), D41.2 (A), D55.2 (A), D69.2 (A), D78.2 (A); no longer D13.2 (A), D28.2 (A), D43.2 (A), D57.2 (A)
- net Col14: now also D27.2 (A), D42.2 (A), D56.2 (A); no longer D14.2 (A), D29.2 (A), D44.2 (A)
- net Col2: now also D15.2 (A), D30.2 (A), D45.2 (A), D58.2 (A), D72.2 (A); no longer D17.2 (A), D2.2 (A), D32.2 (A), D47.2 (A), D60.2 (A), D73.2 (A)
- net Col3: now also D16.2 (A), D2.2 (A), D31.2 (A), D46.2 (A), D59.2 (A); no longer D18.2 (A), D3.2 (A), D33.2 (A), D48.2 (A), D61.2 (A)
- net Col4: now also D17.2 (A), D3.2 (A), D32.2 (A), D47.2 (A), D60.2 (A); no longer D19.2 (A), D34.2 (A), D4.2 (A), D49.2 (A), D62.2 (A)
- net Col5: now also D18.2 (A), D33.2 (A), D4.2 (A), D48.2 (A), D61.2 (A); no longer D20.2 (A), D35.2 (A), D5.2 (A), D50.2 (A), D63.2 (A), D74.2 (A)
- net Col6: now also D19.2 (A), D34.2 (A), D49.2 (A), D5.2 (A), D62.2 (A), D73.2 (A); no longer D21.2 (A), D36.2 (A), D51.2 (A), D6.2 (A), D64.2 (A)
- net Col7: now also D20.2 (A), D35.2 (A), D50.2 (A), D6.2 (A), D63.2 (A); no longer D22.2 (A), D37.2 (A), D52.2 (A), D65.2 (A), D7.2 (A)
- net Col8: now also D21.2 (A), D36.2 (A), D51.2 (A), D64.2 (A), D7.2 (A); no longer D23.2 (A), D38.2 (A), D53.2 (A), D66.2 (A), D8.2 (A)
- net Col9: now also D22.2 (A), D37.2 (A), D52.2 (A), D65.2 (A), D74.2 (A), D8.2 (A); no longer D24.2 (A), D39.2 (A), D54.2 (A), D67.2 (A), D75.2 (A), D9.2 (A)
- net GND: now also PWR_Module1.3 (Pin_3), RotaryEnc1.1 (Pin_1), SW1.6-GND (GND), SW10.6-GND (GND), SW11.6-GND (GND), SW12.6-GND (GND), SW13.6-GND (GND), SW14.6-GND (GND), SW15.6-GND (GND), SW16.6-GND (GND), SW17.6-GND (GND), SW18.6-GND (GND), SW19.6-GND (GND), SW2.6-GND (GND), SW20.6-GND (GND), SW21.6-GND (GND), SW22.6-GND (GND), SW23.6-GND (GND), SW24.6-GND (GND), SW25.6-GND (GND), SW26.6-GND (GND), SW27.6-GND (GND), SW28.6-GND (GND), SW29.6-GND (GND), SW3.6-GND (GND), SW30.6-GND (GND), SW31.6-GND (GND), SW32.6-GND (GND), SW33.6-GND (GND), SW34.6-GND (GND), SW35.6-GND (GND), SW36.6-GND (GND), SW37.6-GND (GND), SW38.6-GND (GND), SW39.6-GND (GND), SW4.6-GND (GND), SW40.6-GND (GND), SW41.6-GND (GND), SW42.6-GND (GND), SW43.6-GND (GND), SW44.6-GND (GND), SW45.6-GND (GND), SW46.6-GND (GND), SW47.6-GND (GND), SW48.6-GND (GND), SW49.6-GND (GND), SW5.6-GND (GND), SW50.6-GND (GND), SW51.6-GND (GND), SW52.6-GND (GND), SW53.6-GND (GND), SW54.6-GND (GND), SW55.6-GND (GND), SW56.6-GND (GND), SW57.6-GND (GND), SW58.6-GND (GND), SW59.6-GND (GND), SW6.6-GND (GND), SW60.6-GND (GND), SW61.6-GND (GND), SW62.6-GND (GND), SW63.6-GND (GND), SW64.6-GND (GND), SW65.6-GND (GND), SW66.6-GND (GND), SW67.6-GND (GND), SW68.6-GND (GND), SW69.6-GND (GND), SW7.6-GND (GND), SW70.6-GND (GND), SW71.6-GND (GND), SW72.6-GND (GND), SW73.6-GND (GND), SW74.6-GND (GND), SW75.6-GND (GND), SW76.6-GND (GND), SW77.6-GND (GND), SW78.6-GND (GND), SW79.6-GND (GND), SW8.6-GND (GND), SW9.6-GND (GND), U3.GND_1 (GND), U3.GND_2 (GND)
- net NEOPIXEL_CONTROLL: now also U3.LV1
- net Row0: now also SW1.1, SW10.1, SW11.1, SW12.1, SW2.1, SW3.1, SW4.1, SW5.1, SW6.1, SW7.1, SW8.1, SW9.1
- net Row1: now also SW13.1, SW14.1, SW15.1, SW16.1, SW17.1, SW18.1, SW19.1, SW20.1, SW21.1, SW22.1, SW23.1, SW24.1, SW25.1, SW26.1, SW27.1
- net Row2: now also SW28.1, SW29.1, SW30.1, SW31.1, SW32.1, SW33.1, SW34.1, SW35.1, SW36.1, SW37.1, SW38.1, SW39.1, SW40.1, SW41.1, SW42.1
- net Row3: now also SW43.1, SW44.1, SW45.1, SW46.1, SW47.1, SW48.1, SW49.1, SW50.1, SW51.1, SW52.1, SW53.1, SW54.1, SW55.1, SW56.1
- net Row4: now also SW57.1, SW58.1, SW59.1, SW60.1, SW61.1, SW62.1, SW63.1, SW64.1, SW65.1, SW66.1, SW67.1, SW68.1, SW69.1
- net Row5: now also SW70.1, SW71.1, SW72.1, SW73.1, SW74.1, SW75.1, SW76.1, SW77.1, SW78.1, SW79.1
- net VCC: now also RotaryEnc1.2 (Pin_2), U3.LV
- net batt_chargesense: now also PWR_Module1.1 (Pin_1)
- net batt_voltage_Pin: now also PWR_Module1.2 (Pin_2)
- net at D52.1 (K): now also SW52.2
- net at D39.1 (K): now also SW39.2
- net at D20.1 (K): now also SW20.2
- net at D68.1 (K): now also SW68.2
- net at D47.1 (K): now also SW47.2
- net at D13.1 (K): now also SW13.2
- net at D62.1 (K): now also SW62.2
- net at D79.1 (K): now also SW79.2
- net at D21.1 (K): now also SW21.2
- net at D40.1 (K): now also SW40.2
- net at D65.1 (K): now also SW65.2
- net at D43.1 (K): now also SW43.2
- net at D23.1 (K): now also SW23.2
- net at D32.1 (K): now also SW32.2
- net at D71.1 (K): now also SW71.2
- net at D19.1 (K): now also SW19.2
- net at D36.1 (K): now also SW36.2
- net at D37.1 (K): now also SW37.2
- net at D61.1 (K): now also SW61.2
- net at D64.1 (K): now also SW64.2
- net at D33.1 (K): now also SW33.2
- net at D29.1 (K): now also SW29.2
- net at D12.1 (K): now also SW12.2
- net at D14.1 (K): now also SW14.2
- net at D55.1 (K): now also SW55.2
- net at D24.1 (K): now also SW24.2
- net at D25.1 (K): now also SW25.2
- net at D72.1 (K): now also SW72.2
- net at D75.1 (K): now also SW75.2
- net at D57.1 (K): now also SW57.2
- net at D1.1 (K): now also SW1.2
- net at D9.1 (K): now also SW9.2
- net at D8.1 (K): now also SW8.2
- net at D17.1 (K): now also SW17.2
- net at D28.1 (K): now also SW28.2
- net at D31.1 (K): now also SW31.2
- net at D51.1 (K): now also SW51.2
- net at D44.1 (K): now also SW44.2
- net at D38.1 (K): now also SW38.2
- net at D5.1 (K): now also SW5.2
- net at D70.1 (K): now also SW70.2
- net at D45.1 (K): now also SW45.2
- net at D59.1 (K): now also SW59.2
- net at D18.1 (K): now also SW18.2
- net at D15.1 (K): now also SW15.2
- net at D63.1 (K): now also SW63.2
- net at D67.1 (K): now also SW67.2
- net at D48.1 (K): now also SW48.2
- net at D66.1 (K): now also SW66.2
- net at D26.1 (K): now also SW26.2
- net at D58.1 (K): now also SW58.2
- net at D60.1 (K): now also SW60.2
- net at D56.1 (K): now also SW56.2
- net at D54.1 (K): now also SW54.2
- net at D73.1 (K): now also SW73.2
- net at D46.1 (K): now also SW46.2
- net at D11.1 (K): now also SW11.2
- net at D10.1 (K): now also SW10.2
- net at D77.1 (K): now also SW77.2
- net at D41.1 (K): now also SW41.2
- net at D6.1 (K): now also SW6.2
- net at D3.1 (K): now also SW3.2
- net at D16.1 (K): now also SW16.2
- net at D49.1 (K): now also SW49.2
- net at D2.1 (K): now also SW2.2
- net at D42.1 (K): now also SW42.2
- net at D78.1 (K): now also SW78.2
- net at D27.1 (K): now also SW27.2
- net at D35.1 (K): now also SW35.2
- net at D50.1 (K): now also SW50.2
- net at D7.1 (K): now also SW7.2
- net at D69.1 (K): now also SW69.2
- net at D74.1 (K): now also SW74.2
- net at D4.1 (K): now also SW4.2
- net ENC_SW: now reaches U5.18 (VN)
- net ENC_SW: now also RotaryEnc1.3 (Pin_3)
- net Vin+: now reaches U5.30 (VIN)
- net Vin+: now also PWR_Module1.4 (Pin_4), SW1.3-VDD (VDD), SW10.3-VDD (VDD), SW11.3-VDD (VDD), SW12.3-VDD (VDD), SW13.3-VDD (VDD), SW14.3-VDD (VDD), SW15.3-VDD (VDD), SW16.3-VDD (VDD), SW17.3-VDD (VDD), SW18.3-VDD (VDD), SW19.3-VDD (VDD), SW2.3-VDD (VDD), SW20.3-VDD (VDD), SW21.3-VDD (VDD), SW22.3-VDD (VDD), SW23.3-VDD (VDD), SW24.3-VDD (VDD), SW25.3-VDD (VDD), SW26.3-VDD (VDD), SW27.3-VDD (VDD), SW28.3-VDD (VDD), SW29.3-VDD (VDD), SW3.3-VDD (VDD), SW30.3-VDD (VDD), SW31.3-VDD (VDD), SW32.3-VDD (VDD), SW33.3-VDD (VDD), SW34.3-VDD (VDD), SW35.3-VDD (VDD), SW36.3-VDD (VDD), SW37.3-VDD (VDD), SW38.3-VDD (VDD), SW39.3-VDD (VDD), SW4.3-VDD (VDD), SW40.3-VDD (VDD), SW41.3-VDD (VDD), SW42.3-VDD (VDD), SW43.3-VDD (VDD), SW44.3-VDD (VDD), SW45.3-VDD (VDD), SW46.3-VDD (VDD), SW47.3-VDD (VDD), SW48.3-VDD (VDD), SW49.3-VDD (VDD), SW5.3-VDD (VDD), SW50.3-VDD (VDD), SW51.3-VDD (VDD), SW52.3-VDD (VDD), SW53.3-VDD (VDD), SW54.3-VDD (VDD), SW55.3-VDD (VDD), SW56.3-VDD (VDD), SW57.3-VDD (VDD), SW58.3-VDD (VDD), SW59.3-VDD (VDD), SW6.3-VDD (VDD), SW60.3-VDD (VDD), SW61.3-VDD (VDD), SW62.3-VDD (VDD), SW63.3-VDD (VDD), SW64.3-VDD (VDD), SW65.3-VDD (VDD), SW66.3-VDD (VDD), SW67.3-VDD (VDD), SW68.3-VDD (VDD), SW69.3-VDD (VDD), SW7.3-VDD (VDD), SW70.3-VDD (VDD), SW71.3-VDD (VDD), SW72.3-VDD (VDD), SW73.3-VDD (VDD), SW74.3-VDD (VDD), SW75.3-VDD (VDD), SW76.3-VDD (VDD), SW77.3-VDD (VDD), SW78.3-VDD (VDD), SW79.3-VDD (VDD), SW8.3-VDD (VDD), SW9.3-VDD (VDD), U3.HV
- net ENC_DT: now reaches U5.6 (RX2)
- net ENC_DT: now also RotaryEnc1.4 (Pin_4)
- net ENC_CLK: now reaches U5.7 (TX2)
- net ENC_CLK: now also RotaryEnc1.5 (Pin_5)
- net at D76.1 (K): now also SW76.2
- net at D53.1 (K): now also SW53.2
- net at D22.1 (K): now also SW22.2
- net at D34.1 (K): now also SW34.2
- net at D30.1 (K): now also SW30.2
- net Col15: no longer names the net of U2.7 (QH)
- net Col15: no longer D70.2 (A)
- new net: SW50.4-DOUT (DO), SW51.5-DIN (DI)
- new net: SW49.4-DOUT (DO), SW50.5-DIN (DI)
- new net: SW64.4-DOUT (DO), SW65.5-DIN (DI)
- new net: SW63.4-DOUT (DO), SW64.5-DIN (DI)
- new net: SW29.4-DOUT (DO), SW30.5-DIN (DI)
- new net: SW28.4-DOUT (DO), SW29.5-DIN (DI)
- new net: SW30.4-DOUT (DO), SW31.5-DIN (DI)
- new net: SW16.4-DOUT (DO), SW17.5-DIN (DI)
- new net: SW15.4-DOUT (DO), SW16.5-DIN (DI)
- new net: SW47.4-DOUT (DO), SW48.5-DIN (DI)
- new net: SW46.4-DOUT (DO), SW47.5-DIN (DI)
- new net: SW56.4-DOUT (DO), SW57.5-DIN (DI)
- new net: SW55.4-DOUT (DO), SW56.5-DIN (DI)
- new net: SW25.4-DOUT (DO), SW26.5-DIN (DI)
- new net: SW24.4-DOUT (DO), SW25.5-DIN (DI)
- new net: SW35.4-DOUT (DO), SW36.5-DIN (DI)
- new net: SW34.4-DOUT (DO), SW35.5-DIN (DI)
- new net: SW61.4-DOUT (DO), SW62.5-DIN (DI)
- new net: SW60.4-DOUT (DO), SW61.5-DIN (DI)
- new net: SW12.4-DOUT (DO), SW13.5-DIN (DI)
- new net: SW11.4-DOUT (DO), SW12.5-DIN (DI)
- new net: SW62.4-DOUT (DO), SW63.5-DIN (DI)
- new net: SW45.4-DOUT (DO), SW46.5-DIN (DI)
- new net: SW44.4-DOUT (DO), SW45.5-DIN (DI)
- new net: SW10.4-DOUT (DO), SW11.5-DIN (DI)
- new net: SW10.5-DIN (DI), SW9.4-DOUT (DO)
- new net: SW37.4-DOUT (DO), SW38.5-DIN (DI)
- new net: SW36.4-DOUT (DO), SW37.5-DIN (DI)
- new net: SW33.4-DOUT (DO), SW34.5-DIN (DI)
- new net: SW73.4-DOUT (DO), SW74.5-DIN (DI)
- new net: SW72.4-DOUT (DO), SW73.5-DIN (DI)
- new net: SW6.4-DOUT (DO), SW7.5-DIN (DI)
- new net: SW5.4-DOUT (DO), SW6.5-DIN (DI)
- new net: SW57.4-DOUT (DO), SW58.5-DIN (DI)
- new net: SW7.4-DOUT (DO), SW8.5-DIN (DI)
- new net: SW23.4-DOUT (DO), SW24.5-DIN (DI)
- new net: SW21.4-DOUT (DO), SW22.5-DIN (DI)
- new net: SW20.4-DOUT (DO), SW21.5-DIN (DI)
- new net: SW66.4-DOUT (DO), SW67.5-DIN (DI)
- new net: SW65.4-DOUT (DO), SW66.5-DIN (DI)
- new net: SW31.4-DOUT (DO), SW32.5-DIN (DI)
- new net: SW40.4-DOUT (DO), SW41.5-DIN (DI)
- new net: SW39.4-DOUT (DO), SW40.5-DIN (DI)
- new net: SW32.4-DOUT (DO), SW33.5-DIN (DI)
- new net: SW13.4-DOUT (DO), SW14.5-DIN (DI)
- new net: SW18.4-DOUT (DO), SW19.5-DIN (DI)
- new net: SW17.4-DOUT (DO), SW18.5-DIN (DI)
- new net: SW26.4-DOUT (DO), SW27.5-DIN (DI)
- new net: SW14.4-DOUT (DO), SW15.5-DIN (DI)
- new net: SW41.4-DOUT (DO), SW42.5-DIN (DI)
- new net: SW78.4-DOUT (DO), SW79.5-DIN (DI)
- new net: SW71.4-DOUT (DO), SW72.5-DIN (DI)
- new net: SW42.4-DOUT (DO), SW43.5-DIN (DI)
- new net: SW53.4-DOUT (DO), SW54.5-DIN (DI)
- new net: SW52.4-DOUT (DO), SW53.5-DIN (DI)
- new net: SW8.4-DOUT (DO), SW9.5-DIN (DI)
- new net: SW48.4-DOUT (DO), SW49.5-DIN (DI)
- new net: SW75.4-DOUT (DO), SW76.5-DIN (DI)
- new net: SW74.4-DOUT (DO), SW75.5-DIN (DI)
- new net: SW4.4-DOUT (DO), SW5.5-DIN (DI)
- new net: SW3.4-DOUT (DO), SW4.5-DIN (DI)
- new net: SW67.4-DOUT (DO), SW68.5-DIN (DI)
- new net: SW19.4-DOUT (DO), SW20.5-DIN (DI)
- new net: SW22.4-DOUT (DO), SW23.5-DIN (DI)
- new net: SW51.4-DOUT (DO), SW52.5-DIN (DI)
- new net: SW2.4-DOUT (DO), SW3.5-DIN (DI)
- new net: SW1.4-DOUT (DO), SW2.5-DIN (DI)
- new net: SW68.4-DOUT (DO), SW69.5-DIN (DI)
- new net: SW59.4-DOUT (DO), SW60.5-DIN (DI)
- new net: SW70.4-DOUT (DO), SW71.5-DIN (DI)
- new net: SW54.4-DOUT (DO), SW55.5-DIN (DI)
- new net: SW58.4-DOUT (DO), SW59.5-DIN (DI)
- new net: SW43.4-DOUT (DO), SW44.5-DIN (DI)
- new net: SW38.4-DOUT (DO), SW39.5-DIN (DI)
- new net: SW76.4-DOUT (DO), SW77.5-DIN (DI)
- new net: SW27.4-DOUT (DO), SW28.5-DIN (DI)
- new net: SW77.4-DOUT (DO), SW78.5-DIN (DI)
- new net: SW69.4-DOUT (DO), SW70.5-DIN (DI)
- new net NEOPIXEL5VData: SW1.5-DIN (DI), U3.HV1
- no-connect marks 0 -> 10
Other:
- note added: "Display"
- note added: "ESP 32"
- note added: "Logic Level Shifter"
- note added: "Power Module input"
- note added: "Rotary Encoder"
- note added: "Shift register"
- note added: "Slider Potentiometer"
- title: (none) -> ESP 32 Keyboard matrix and controller
- moved on the sheet: C1, C2, Dsp1, R1, R2, R3, R4, R5, R6, R7, S1, S2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
